Commit message: add mapping

File: farmbot_description/urdf/diffbot_description.urdf.xacro (robot description, xacro)
@@ -14,4 +14,10 @@
   <xacro:property name="caster_wheel_radius" value="0.015" />
   <xacro:property name="z_offset" value="-${base_height/2}" /> <!-- Space btw top of beam and the each joint -->
+   <link name="base_footprint"></link>
+   <joint name="base_footprint_joint" type="fixed">
+    <parent link="base_footprint"/>
+    <child link="base_link"/>
+    <origin xyz="0 0 0" rpy="0 0 0"/>
+   </joint>
   <!-- Base Link -->
   <link name="base_link">
